Commit message: feat(web): use kuavo biped_v3_arm as test_arm and fix prod loading
- Repackage test_arm from biped_s56 biped_v3_arm.urdf with real STL meshes
- Add test-arm-loader; wire load test_arm button and PROD default model
- Restore URDF folder/ZIP picker as native select dropdown
- Keep simple_test_arm.urdf fixture for unit tests

File: public/robots/test_arm.urdf (robot description, URDF)
Before this commit: robot test_arm, 8 links, 7 joints
Links:
- removed link ee_link
- removed link link1
- removed link link2
- removed link link3
- removed link link4
- removed link link5
- removed link world
- added link waist_yaw_link, mass 20.63616; visual mesh filename=test_arm/meshes/waist_yaw.STL
- added link zarm_l1_link, mass 0.94521; visual mesh filename=test_arm/meshes/l_arm_pitch.STL
- added link zarm_l2_link, mass 0.41921; visual mesh filename=test_arm/meshes/l_arm_roll.STL
- added link zarm_l3_link, mass 1.78857; visual mesh filename=test_arm/meshes/l_arm_yaw.STL
- added link zarm_l4_link, mass 0.63149; visual mesh filename=test_arm/meshes/l_forearm.STL
- added link zarm_l5_link, mass 0.60828; visual mesh filename=test_arm/meshes/l_hand_yaw.STL
- added link zarm_l6_link, mass 0.50616; visual mesh filename=test_arm/meshes/l_hand_roll.STL
- added link zarm_l7_end_effector
- added link zarm_l7_link, mass 0.7374; visual mesh filename=test_arm/meshes/l_hand_pitch_nohand.STL
- added link zarm_l7_virtual_thumb_link; collision sphere radius=0.005
- added link zarm_r1_link, mass 0.92947; visual mesh filename=test_arm/meshes/r_arm_pitch.STL
- added link zarm_r2_link, mass 0.41523; visual mesh filename=test_arm/meshes/r_arm_roll.STL
- added link zarm_r3_link, mass 1.78473; visual mesh filename=test_arm/meshes/r_arm_yaw.STL
- added link zarm_r4_link, mass 0.63548; visual mesh filename=test_arm/meshes/r_forearm.STL
- added link zarm_r5_link, mass 0.61021; visual mesh filename=test_arm/meshes/r_hand_yaw.STL
- added link zarm_r6_link, mass 0.53821; visual mesh filename=test_arm/meshes/r_hand_roll.STL
- added link zarm_r7_end_effector
- added link zarm_r7_link, mass 0.7374; visual mesh filename=test_arm/meshes/r_hand_pitch_nohand.STL
- added link zarm_r7_virtual_thumb_link; collision sphere radius=0.005
- link base_link: mass 1.0 -> 7.06405; geometry visual mesh filename=test_arm/meshes/torso.STL
Joints:
- removed joint ee_joint
- removed joint joint1
- removed joint joint2
- removed joint joint3
- removed joint joint4
- removed joint joint5
- removed joint world_to_base
- added joint waist_yaw_joint: type fixed, parent base_link, child waist_yaw_link, origin xyz=0 0 0.1114 rpy=0 0 0, axis 0 0 1, limit lower=-3.14159 upper=3.14159 effort=102.0 velocity=8.7
- added joint zarm_l1_joint: type revolute, parent waist_yaw_link, child zarm_l1_link, origin xyz=-0.003 0.2527 0.283 rpy=0 0 0, axis 0 1 0, limit lower=-3.14159265358979 upper=1.5707963267949 effort=66.0 velocity=18.8
- added joint zarm_l2_joint: type revolute, parent zarm_l1_link, child zarm_l2_link, origin xyz=0 0 0 rpy=0 0 0, axis 1 0 0, limit lower=-0.349065850398866 upper=3.49065850398866 effort=75.0 velocity=8.0
- added joint zarm_l3_joint: type revolute, parent zarm_l2_link, child zarm_l3_link, origin xyz=0 0 0 rpy=0 0 0, axis 0 0 1, limit lower=-1.48352986419518 upper=1.48352986419518 effort=57.0 velocity=7.5
- added joint zarm_l4_joint: type revolute, parent zarm_l3_link, child zarm_l4_link, origin xyz=0.02 0 -0.2837 rpy=0 0 0, axis 0 1 0, limit lower=-2.61799387799149 upper=0.0 effort=75.0 velocity=8.0
- added joint zarm_l5_joint: type revolute, parent zarm_l4_link, child zarm_l5_link, origin xyz=-0.02 0 -0.1201 rpy=0 0 0, axis 0 0 1, limit lower=-1.5707963267949 upper=1.5707963267949 effort=14.1 velocity=17.5
- added joint zarm_l6_joint: type revolute, parent zarm_l5_link, child zarm_l6_link, origin xyz=0.0 0 -0.114 rpy=0 0 0, axis 1 0 0, limit lower=-1.30899693899575 upper=0.698131700797732 effort=14.1 velocity=17.5
- added joint zarm_l7_end_effector_joint: type fixed, parent zarm_l7_link, child zarm_l7_end_effector, origin xyz=0 0.0 -0.17 rpy=0 0 0
- added joint zarm_l7_joint: type revolute, parent zarm_l6_link, child zarm_l7_link, origin xyz=0 0 -0.021 rpy=0 0 0, axis 0 1 0, limit lower=-0.698131700797732 upper=0.698131700797732 effort=14.1 velocity=17.5
- added joint zarm_l7_virtual_thumb_joint_ee: type fixed, parent zarm_l7_end_effector, child zarm_l7_virtual_thumb_link, origin xyz=0.15 0 0 rpy=0 0 0
- added joint zarm_r1_joint: type revolute, parent waist_yaw_link, child zarm_r1_link, origin xyz=-0.003 -0.2527 0.283 rpy=0 0 0, axis 0 1 0, limit lower=-3.14159265358979 upper=1.5707963267949 effort=66.0 velocity=18.8
- added joint zarm_r2_joint: type revolute, parent zarm_r1_link, child zarm_r2_link, origin xyz=0 0 0 rpy=0 0 0, axis 1 0 0, limit lower=-3.49065850398866 upper=0.349065850398866 effort=75.0 velocity=8.0
- added joint zarm_r3_joint: type revolute, parent zarm_r2_link, child zarm_r3_link, origin xyz=0 0 0 rpy=0 0 0, axis 0 0 1, limit lower=-1.48352986419518 upper=1.48352986419518 effort=57.0 velocity=7.5
- added joint zarm_r4_joint: type revolute, parent zarm_r3_link, child zarm_r4_link, origin xyz=0.02 0 -0.2837 rpy=0 0 0, axis 0 1 0, limit lower=-2.61799387799149 upper=0.0 effort=75.0 velocity=8.0
- added joint zarm_r5_joint: type revolute, parent zarm_r4_link, child zarm_r5_link, origin xyz=-0.02 0 -0.1201 rpy=0 0 0, axis 0 0 1, limit lower=-1.5707963267949 upper=1.5707963267949 effort=14.1 velocity=17.5
- added joint zarm_r6_joint: type revolute, parent zarm_r5_link, child zarm_r6_link, origin xyz=0.0 0 -0.114 rpy=0 0 0, axis 1 0 0, limit lower=-0.698131700797732 upper=1.30899693899575 effort=14.1 velocity=17.5
- added joint zarm_r7_end_effector_joint: type fixed, parent zarm_r7_link, child zarm_r7_end_effector, origin xyz=0 0.0 -0.17 rpy=0 0 0
- added joint zarm_r7_joint: type revolute, parent zarm_r6_link, child zarm_r7_link, origin xyz=0.0 0 -0.021 rpy=0 0 0, axis 0 1 0, limit lower=-0.698131700797732 upper=0.698131700797732 effort=14.1 velocity=17.5
- added joint zarm_r7_virtual_thumb_joint_ee: type fixed, parent zarm_r7_end_effector, child zarm_r7_virtual_thumb_link, origin xyz=0.15 0 0 rpy=0 0 0

File: public/robots/test_arm/urdf/test_arm.urdf (robot description, URDF)
Before this commit: robot test_arm, 8 links, 7 joints
Links:
- removed link ee_link
- removed link link1
- removed link link2
- removed link link3
- removed link link4
- removed link link5
- removed link world
- added link waist_yaw_link, mass 20.63616; visual mesh filename=../meshes/waist_yaw.STL
- added link zarm_l1_link, mass 0.94521; visual mesh filename=../meshes/l_arm_pitch.STL
- added link zarm_l2_link, mass 0.41921; visual mesh filename=../meshes/l_arm_roll.STL
- added link zarm_l3_link, mass 1.78857; visual mesh filename=../meshes/l_arm_yaw.STL
- added link zarm_l4_link, mass 0.63149; visual mesh filename=../meshes/l_forearm.STL
- added link zarm_l5_link, mass 0.60828; visual mesh filename=../meshes/l_hand_yaw.STL
- added link zarm_l6_link, mass 0.50616; visual mesh filename=../meshes/l_hand_roll.STL
- added link zarm_l7_end_effector
- added link zarm_l7_link, mass 0.7374; visual mesh filename=../meshes/l_hand_pitch_nohand.STL
- added link zarm_l7_virtual_thumb_link; collision sphere radius=0.005
- added link zarm_r1_link, mass 0.92947; visual mesh filename=../meshes/r_arm_pitch.STL
- added link zarm_r2_link, mass 0.41523; visual mesh filename=../meshes/r_arm_roll.STL
- added link zarm_r3_link, mass 1.78473; visual mesh filename=../meshes/r_arm_yaw.STL
- added link zarm_r4_link, mass 0.63548; visual mesh filename=../meshes/r_forearm.STL
- added link zarm_r5_link, mass 0.61021; visual mesh filename=../meshes/r_hand_yaw.STL
- added link zarm_r6_link, mass 0.53821; visual mesh filename=../meshes/r_hand_roll.STL
- added link zarm_r7_end_effector
- added link zarm_r7_link, mass 0.7374; visual mesh filename=../meshes/r_hand_pitch_nohand.STL
- added link zarm_r7_virtual_thumb_link; collision sphere radius=0.005
- link base_link: mass 1.0 -> 7.06405; geometry visual mesh filename=../meshes/torso.STL
Joints:
- removed joint ee_joint
- removed joint joint1
- removed joint joint2
- removed joint joint3
- removed joint joint4
- removed joint joint5
- removed joint world_to_base
- added joint waist_yaw_joint: type fixed, parent base_link, child waist_yaw_link, origin xyz=0 0 0.1114 rpy=0 0 0, axis 0 0 1, limit lower=-3.14159 upper=3.14159 effort=102.0 velocity=8.7
- added joint zarm_l1_joint: type revolute, parent waist_yaw_link, child zarm_l1_link, origin xyz=-0.003 0.2527 0.283 rpy=0 0 0, axis 0 1 0, limit lower=-3.14159265358979 upper=1.5707963267949 effort=66.0 velocity=18.8
- added joint zarm_l2_joint: type revolute, parent zarm_l1_link, child zarm_l2_link, origin xyz=0 0 0 rpy=0 0 0, axis 1 0 0, limit lower=-0.349065850398866 upper=3.49065850398866 effort=75.0 velocity=8.0
- added joint zarm_l3_joint: type revolute, parent zarm_l2_link, child zarm_l3_link, origin xyz=0 0 0 rpy=0 0 0, axis 0 0 1, limit lower=-1.48352986419518 upper=1.48352986419518 effort=57.0 velocity=7.5
- added joint zarm_l4_joint: type revolute, parent zarm_l3_link, child zarm_l4_link, origin xyz=0.02 0 -0.2837 rpy=0 0 0, axis 0 1 0, limit lower=-2.61799387799149 upper=0.0 effort=75.0 velocity=8.0
- added joint zarm_l5_joint: type revolute, parent zarm_l4_link, child zarm_l5_link, origin xyz=-0.02 0 -0.1201 rpy=0 0 0, axis 0 0 1, limit lower=-1.5707963267949 upper=1.5707963267949 effort=14.1 velocity=17.5
- added joint zarm_l6_joint: type revolute, parent zarm_l5_link, child zarm_l6_link, origin xyz=0.0 0 -0.114 rpy=0 0 0, axis 1 0 0, limit lower=-1.30899693899575 upper=0.698131700797732 effort=14.1 velocity=17.5
- added joint zarm_l7_end_effector_joint: type fixed, parent zarm_l7_link, child zarm_l7_end_effector, origin xyz=0 0.0 -0.17 rpy=0 0 0
- added joint zarm_l7_joint: type revolute, parent zarm_l6_link, child zarm_l7_link, origin xyz=0 0 -0.021 rpy=0 0 0, axis 0 1 0, limit lower=-0.698131700797732 upper=0.698131700797732 effort=14.1 velocity=17.5
- added joint zarm_l7_virtual_thumb_joint_ee: type fixed, parent zarm_l7_end_effector, child zarm_l7_virtual_thumb_link, origin xyz=0.15 0 0 rpy=0 0 0
- added joint zarm_r1_joint: type revolute, parent waist_yaw_link, child zarm_r1_link, origin xyz=-0.003 -0.2527 0.283 rpy=0 0 0, axis 0 1 0, limit lower=-3.14159265358979 upper=1.5707963267949 effort=66.0 velocity=18.8
- added joint zarm_r2_joint: type revolute, parent zarm_r1_link, child zarm_r2_link, origin xyz=0 0 0 rpy=0 0 0, axis 1 0 0, limit lower=-3.49065850398866 upper=0.349065850398866 effort=75.0 velocity=8.0
- added joint zarm_r3_joint: type revolute, parent zarm_r2_link, child zarm_r3_link, origin xyz=0 0 0 rpy=0 0 0, axis 0 0 1, limit lower=-1.48352986419518 upper=1.48352986419518 effort=57.0 velocity=7.5
- added joint zarm_r4_joint: type revolute, parent zarm_r3_link, child zarm_r4_link, origin xyz=0.02 0 -0.2837 rpy=0 0 0, axis 0 1 0, limit lower=-2.61799387799149 upper=0.0 effort=75.0 velocity=8.0
- added joint zarm_r5_joint: type revolute, parent zarm_r4_link, child zarm_r5_link, origin xyz=-0.02 0 -0.1201 rpy=0 0 0, axis 0 0 1, limit lower=-1.5707963267949 upper=1.5707963267949 effort=14.1 velocity=17.5
- added joint zarm_r6_joint: type revolute, parent zarm_r5_link, child zarm_r6_link, origin xyz=0.0 0 -0.114 rpy=0 0 0, axis 1 0 0, limit lower=-0.698131700797732 upper=1.30899693899575 effort=14.1 velocity=17.5
- added joint zarm_r7_end_effector_joint: type fixed, parent zarm_r7_link, child zarm_r7_end_effector, origin xyz=0 0.0 -0.17 rpy=0 0 0
- added joint zarm_r7_joint: type revolute, parent zarm_r6_link, child zarm_r7_link, origin xyz=0.0 0 -0.021 rpy=0 0 0, axis 0 1 0, limit lower=-0.698131700797732 upper=0.698131700797732 effort=14.1 velocity=17.5
- added joint zarm_r7_virtual_thumb_joint_ee: type fixed, parent zarm_r7_end_effector, child zarm_r7_virtual_thumb_link, origin xyz=0.15 0 0 rpy=0 0 0
